File: kicad/EllaFi-PCB.kicad_sch (KiCad schematic)
At the start: 26 parts, among them J1 Conn_01x04_Socket, J2 Conn_01x03, J3 PJ-002AH, J4 Conn_01x22_Socket, J5 Conn_01x22_Socket, Q1 AOD4184A, SW1 OS102011MS2QN1, U1 FOD817S, U3 MPM3620AGQV-Z

Commit message: kicad: whole-board validation suite + fix 4 sim-found defects
New kicad/sim/board/ (./run_all.sh): pad-polarity checker (board vs
datasheet intent), sim-sync checker (SPICE model vs fresh netlist
export), 11 ngspice scenario benches + 60-trial Monte Carlo.

Defects the suite found, fixed in schematic+PCB:
- D4 saw 7V reverse (5V-max LED) whenever Q1 off -> moved with R4 to
  the gate side; also now clamps GPIO14 during boot vs pullup panels
- reversed adapter put -12V on the buck -> D6 1.5SMC18CA (bidir) ->
  1.5SMC18A (unidir), band to 12V rail; clamps -0.8V, F1 trips
- D1 coin-line TVS installed backwards (band on GND -> would clamp
  the coin line at 0.7V; dead coin input) -> flipped
- low-CTR/aged optos left GPIO4 above the 0.825V logic-low ceiling
  (~5% of builds) -> R1 1k->2.2k, R5 220->1k (4.7k rejected: too slow
  recovering from coupled noise bursts)

globals.h: J2.2 3-wire panel TODO closed with the sim verdict; stale
IRLZ44N/10k comment facts corrected. Findings + lessons recorded in
memory/hardware_notes.md. ERC 0, DRC 0, suite ALL PASS.

Co-Authored-By: Claude Fable 5 <noreply@anthropic.com>
Parts:
- C1: DigiKey_PN 493-14973-ND -> 1276-2397-1-ND; Mfg_PN UEP1E101MPD -> CL21A106KACLRNC
- C2: DigiKey_PN 493-14973-ND -> 1276-7092-1-ND; Mfg_PN UEP1E101MPD -> CL21A226KOQNNNG
- D1: DigiKey_PN P6KE6.8ALFCT-ND -> P6SMB6.8ALFCT-ND; LCSC P6KE6.8A -> P6SMB6.8A; Mfg_PN P6KE6.8A -> P6SMB6.8A
- D3: DigiKey_PN 732-5006-ND -> AP3216SURCK-ND; Mfg_PN 151031SS06000 -> AP3216SURCK
- D4: DigiKey_PN 732-5010-ND -> AP3216SYCK-ND; Mfg_PN 151031YS06000 -> AP3216SYCK
- D5: DigiKey_PN 732-5008-ND -> AP3216SGCK-ND; Mfg_PN 151031VS06000 -> AP3216SGCK
- D6: value 1.5SMC18CA -> 1.5SMC18A; DigiKey_PN (none) -> 1.5SMC18ABB-ND; Mfg_PN (none) -> 1.5SMC18A
- F1: value miniSMDC150F -> MINISMDC150F/16-2; DigiKey_PN (none) -> MINISMDC150F/16-2CT-ND; Mfg_PN (none) -> MINISMDC150F/16-2
- Q1: DigiKey_PN IRLZ44NPBF-ND -> 785-1221-1-ND; Mfg_PN IRLZ44NPBF -> AOD4184A
- R1: value 1k -> 2.2k; DigiKey_PN MF0207FRE52-1K-ND -> 311-2.20KCRCT-ND; Mfg_PN MF0207FRE52-1K -> RC0805FR-072K2L
- R2, R4: DigiKey_PN 220QBK-ND -> 311-220CRCT-ND; Mfg_PN CFR-25JB-52-220R -> RC0805FR-07220RL
- R3: DigiKey_PN 330QBK-ND -> 311-330CRCT-ND; Mfg_PN CFR-25JB-52-330R -> RC0805FR-07330RL
- R5: value 220 -> 1k; DigiKey_PN 220QBK-ND -> 311-1.00KCRCT-ND; Mfg_PN CFR-25JB-52-220R -> RC0805FR-071KL
- R6: DigiKey_PN MF0207FRE52-10K-ND -> 311-10.0KCRCT-ND; Mfg_PN MF0207FRE52-10K -> RC0805FR-0710KL
- R7, R9: DigiKey_PN (none) -> 311-100KLRCT-ND; Mfg_PN (none) -> RC0402FR-07100KL
- R8: DigiKey_PN (none) -> 311-19.1KLRCT-ND; Mfg_PN (none) -> RC0402FR-0719K1L
- U1: DigiKey_PN FOD817-ND -> FOD817S-ND; Mfg_PN FOD817 -> FOD817S
- U3: DigiKey_PN (none) -> MPM3620AGQV-Z-ND; Mfg_PN (none) -> MPM3620AGQV-Z
Connections:
- net 5V: no longer R4.2
- net GND: now also D1.2 (A2), D6.2 (A2), R4.2; no longer D1.1 (A1), D6.1 (A1)
- net GPIO14: now also D4.2 (A)
- net at J1.3 (Pin_3), Q1.2 (D), SW1.1 (A): no longer D4.1 (K)
- net at C1.1, F1.2, J1.1 (Pin_1)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: now also D6.1 (A1); no longer D6.2 (A2)
- net at R4.1: now also D4.1 (K); no longer D4.2 (A)
- net at J1.2 (Pin_2), U1.2: now also D1.1 (A1); no longer D1.2 (A2)
Other:
- moved on the sheet: D1, D4, D6, R4

Commit message: kicad: order-time BOM fixes — D6 DigiKey PN corrected (118-1.5SMC18ACT-ND, verified in stock), J2 Phoenix 1715857 -> generic WJ500V-5.08-3P (KF301 family, JLC-stocked, same 5.08mm 3-pos footprint)
Co-Authored-By: Claude Fable 5 <noreply@anthropic.com>
Parts:
- D6: DigiKey_PN 1.5SMC18ABB-ND -> 118-1.5SMC18ACT-ND
- J2: DigiKey_PN 277-1976-ND -> (none); Mfg_PN 1715857 -> WJ500V-5.08-3P
Changed lines of the file:
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@@
 			)
 		)
-		(property "DigiKey_PN" "277-1976-ND"
+		(property "DigiKey_PN" ""
 			(at 68.58 90.17 0)
 			(hide yes)
@@
 			)
 		)
-		(property "Mfg_PN" "1715857"
+		(property "Mfg_PN" "WJ500V-5.08-3P"
 			(at 68.58 90.17 0)
 			(hide yes)
@@
 			)
 		)
-		(property "DigiKey_PN" "1.5SMC18ABB-ND"
+		(property "DigiKey_PN" "118-1.5SMC18ACT-ND"
 			(at 50.8 38.1 0)
 			(hide yes)

Commit message: kicad: LCSC part numbers as schematic fields + one-command JLC export
Every symbol carries an LCSC field (22 pinned from the verified JLC
order; J1/J2/J4/J5 pending final connector picks). Mfg_PN updated on the
6 lines ordered as substitutes: caps -> in-stock Samsung equivalents,
LEDs -> Lite-On LTST-C150 K-RKT/YKT/KGKT (matcher had offered green for
the yellow), U1 -> LTV-817S-TA1-B (CTR-binned 130-260%: removes the
low-CTR tail from the Monte Carlo analysis at the supply level).
export_jlc.py regenerates gerbers+BOM+CPL from these fields.

Co-Authored-By: Claude Fable 5 <noreply@anthropic.com>
Parts:
- C1: LCSC (none) -> C15850; Mfg_PN CL21A106KACLRNC -> CL21A106KAYNNNE
- C2: LCSC (none) -> C98190; Mfg_PN CL21A226KOQNNNG -> CL21A226MOQNNNE
- D1: LCSC P6SMB6.8A -> C19077595
- D3: LCSC (none) -> C125086; Mfg_PN AP3216SURCK -> LTST-C150KRKT
- D4: LCSC (none) -> C125089; Mfg_PN AP3216SYCK -> LTST-C150YKT
- D5: LCSC (none) -> C125085; Mfg_PN AP3216SGCK -> LTST-C150KGKT
- D6: LCSC (none) -> C223925
- F1: LCSC (none) -> C315955
- J3: LCSC (none) -> C2961147
- Q1: LCSC (none) -> C99124
- R1: LCSC (none) -> C114561
- R2, R4: LCSC (none) -> C114519
- R3: LCSC (none) -> C105878
- R5: LCSC (none) -> C95781
- R6: LCSC (none) -> C84376
- R7, R9: LCSC (none) -> C60491
- R8: LCSC (none) -> C138042
- SW1: LCSC (none) -> C221829
- U1: LCSC (none) -> C109226; Mfg_PN FOD817S -> LTV-817S-TA1-B
- U3: LCSC (none) -> C529064

Commit message: kicad: J2 pinned to KF301-5.0-3P / C474882 (in-stock 5.08mm 3P screw terminal)
Co-Authored-By: Claude Fable 5 <noreply@anthropic.com>
Parts:
- J2: LCSC (none) -> C474882; Mfg_PN WJ500V-5.08-3P -> KF301-5.0-3P
Changed lines of the file:
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@@
 			)
 		)
-		(property "Mfg_PN" "WJ500V-5.08-3P"
+		(property "Mfg_PN" "KF301-5.0-3P"
 			(at 68.58 90.17 0)
 			(hide yes)
@@
 			)
 		)
-		(property "LCSC" ""
+		(property "LCSC" "C474882"
 			(at 68.58 90.17 0)
 			(hide yes)

Commit message: kicad: pin J1/J4/J5 sockets (Sullins PPPC0/221LFBN-RC) — BOM now fully specified
All 26 parts carry LCSC numbers; export_jlc.py reports 'fully pinned'.
Sockets go via JLC Global Sourcing (7-15 days); U1 opto and everything
else in-stock. Next order needs no re-matching.

Co-Authored-By: Claude Fable 5 <noreply@anthropic.com>
Parts:
- J1: LCSC (none) -> C6629381
- J4, J5: LCSC (none) -> C6256235
Changed lines of the file:
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@@
 			)
 		)
-		(property "LCSC" ""
+		(property "LCSC" "C6256235"
 			(at 156.21 134.62 0)
 			(hide yes)
@@
 			)
 		)
-		(property "LCSC" ""
+		(property "LCSC" "C6256235"
 			(at 125.73 134.62 0)
 			(hide yes)
@@
 			)
 		)
-		(property "LCSC" ""
+		(property "LCSC" "C6629381"
 			(at 68.58 59.69 0)
 			(hide yes)

Commit message: opto finalized: TLP185(GR-TPL,SE) / C128776 (EL357N out of stock)
As-ordered part after the EL357N sold out in every bin. Toshiba TLP185,
GR CTR bin 100-300%, SOP-4-2.54mm (JLC confirmed footprint match),
identical pinout. Sim re-run for the GR CTR range: ALL PASS (coin lows
0.054V at CTR 3.0/1.0/0.6, Monte Carlo 60/60).

Honest finding: TLP185 LED reverse rating VR=5V (vs 6V for 817/EL357N).
The 12V-short-onto-coin-wire fault drives the LED to 5.5V reverse, 0.5V
over — fault-only, transient, F1 trips, low risk on this batch. Logged
as a rev-B item (coin-line reverse clamp) in TODO.md + README; opto_vrev
bench now INFO. Schematic U1 + fab BOM updated to C128776.

Co-Authored-By: Claude Fable 5 <noreply@anthropic.com>
Parts:
- U1: value FOD817S -> TLP185(GR-TPL,SE); LCSC C109226 -> C128776; Mfg_PN LTV-817S-TA1-B -> TLP185(GR-TPL,SE)
Changed lines of the file:
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@@
 			)
 		)
-		(property "Value" "FOD817S"
+		(property "Value" "TLP185(GR-TPL,SE)"
 			(at 189.23 111.76 0)
 			(show_name no)
@@
 			)
 		)
-		(property "Mfg_PN" "LTV-817S-TA1-B"
+		(property "Mfg_PN" "TLP185(GR-TPL,SE)"
 			(at 189.23 118.11 0)
 			(hide yes)
@@
 			)
 		)
-		(property "LCSC" "C109226"
+		(property "LCSC" "C128776"
 			(at 189.23 118.11 0)
 			(hide yes)
